File: pcb_src/ILM139C_matrix/ILM139C.kicad_sch (KiCad schematic)
At the start: 119 parts, among them CN3 AXE640124D, CN4 AXE640124D, U10 XL-B1010RGBT-HF, U100 XL-B1010RGBT-HF, U101 XL-B1010RGBT-HF, U102 XL-B1010RGBT-HF, U103 XL-B1010RGBT-HF, U104 XL-B1010RGBT-HF, U105 XL-B1010RGBT-HF, U106 XL-B1010RGBT-HF, U107 XL-B1010RGBT-HF, U108 XL-B1010RGBT-HF, U109 XL-B1010RGBT-HF, U11 XL-B1010RGBT-HF, U110 XL-B1010RGBT-HF, U111 XL-B1010RGBT-HF, U112 XL-B1010RGBT-HF, U113 XL-B1010RGBT-HF, U114 XL-B1010RGBT-HF, U115 XL-B1010RGBT-HF, U116 XL-B1010RGBT-HF, U117 XL-B1010RGBT-HF, U118 XL-B1010RGBT-HF, U12 XL-B1010RGBT-HF, U13 XL-B1010RGBT-HF, U14 XL-B1010RGBT-HF, U15 XL-B1010RGBT-HF, U16 XL-B1010RGBT-HF, U17 XL-B1010RGBT-HF, U18 XL-B1010RGBT-HF, U19 XL-B1010RGBT-HF, U2 XL-B1010RGBT-HF, U20 XL-B1010RGBT-HF, U21 XL-B1010RGBT-HF, U22 XL-B1010RGBT-HF, U23 XL-B1010RGBT-HF, U24 XL-B1010RGBT-HF, U25 XL-B1010RGBT-HF, U26 XL-B1010RGBT-HF, U27 XL-B1010RGBT-HF, U28 XL-B1010RGBT-HF, U29 XL-B1010RGBT-HF, U3 XL-B1010RGBT-HF, U30 XL-B1010RGBT-HF, U31 XL-B1010RGBT-HF, U32 XL-B1010RGBT-HF, U33 XL-B1010RGBT-HF, U34 XL-B1010RGBT-HF, U35 XL-B1010RGBT-HF, U36 XL-B1010RGBT-HF, U37 XL-B1010RGBT-HF, U38 XL-B1010RGBT-HF, U39 XL-B1010RGBT-HF, U4 XL-B1010RGBT-HF, U40 XL-B1010RGBT-HF, U41 XL-B1010RGBT-HF, U42 XL-B1010RGBT-HF, U43 XL-B1010RGBT-HF, U44 XL-B1010RGBT-HF, U45 XL-B1010RGBT-HF, U46 XL-B1010RGBT-HF, U47 XL-B1010RGBT-HF, U48 XL-B1010RGBT-HF, U49 XL-B1010RGBT-HF, U5 XL-B1010RGBT-HF, U50 XL-B1010RGBT-HF, U51 XL-B1010RGBT-HF, U52 XL-B1010RGBT-HF, U53 XL-B1010RGBT-HF, U54 XL-B1010RGBT-HF, U55 XL-B1010RGBT-HF, U56 XL-B1010RGBT-HF, U57 XL-B1010RGBT-HF, U58 XL-B1010RGBT-HF, U59 XL-B1010RGBT-HF, U6 XL-B1010RGBT-HF, U60 XL-B1010RGBT-HF, U61 XL-B1010RGBT-HF, U62 XL-B1010RGBT-HF, U63 XL-B1010RGBT-HF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

Commit message: Matrix design, visual
Connections:
- net GND: now reaches CN3.10
- net GND: now also CN3.11, CN3.12, CN3.13, CN3.14, CN3.15, CN3.16, CN3.17, CN3.18, CN3.19, CN3.20, CN3.4, CN3.5, CN3.6, CN3.7, CN3.8, CN3.9, CN4.24, CN4.25, CN4.26, CN4.27, CN4.29, CN4.30, CN4.31, CN4.32, CN4.5, CN4.6, CN4.7
Other:
- company: (none) -> EDrTech d.o.o.
- title: (none) -> ILM139C RGB LED matrix
- moved on the sheet: CN3, CN4, U10, U100, U101, U102, U103, U104, U105, U106, U107, U108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
