File: pcb_src/ILM139C_matrix/ILM139C.kicad_pcb (KiCad board)
At the start: 4 copper layers, 26 x 18 mm, 119 parts, among them CN3 AXE640124D, CN4 AXE640124D, U10 XL-B1010RGBT-HF, U100 XL-B1010RGBT-HF, U101 XL-B1010RGBT-HF, U102 XL-B1010RGBT-HF, U103 XL-B1010RGBT-HF, U104 XL-B1010RGBT-HF, U105 XL-B1010RGBT-HF, U106 XL-B1010RGBT-HF, U107 XL-B1010RGBT-HF, U108 XL-B1010RGBT-HF, U109 XL-B1010RGBT-HF, U11 XL-B1010RGBT-HF, U110 XL-B1010RGBT-HF, U111 XL-B1010RGBT-HF, U112 XL-B1010RGBT-HF, U113 XL-B1010RGBT-HF, U114 XL-B1010RGBT-HF, U115 XL-B1010RGBT-HF, U116 XL-B1010RGBT-HF, U117 XL-B1010RGBT-HF, U118 XL-B1010RGBT-HF, U12 XL-B1010RGBT-HF, U13 XL-B1010RGBT-HF, U14 XL-B1010RGBT-HF, U15 XL-B1010RGBT-HF, U16 XL-B1010RGBT-HF, U17 XL-B1010RGBT-HF, U18 XL-B1010RGBT-HF, U19 XL-B1010RGBT-HF, U2 XL-B1010RGBT-HF, U20 XL-B1010RGBT-HF, U21 XL-B1010RGBT-HF, U22 XL-B1010RGBT-HF, U23 XL-B1010RGBT-HF, U24 XL-B1010RGBT-HF, U25 XL-B1010RGBT-HF, U26 XL-B1010RGBT-HF, U27 XL-B1010RGBT-HF, U28 XL-B1010RGBT-HF, U29 XL-B1010RGBT-HF, U3 XL-B1010RGBT-HF, U30 XL-B1010RGBT-HF, U31 XL-B1010RGBT-HF, U32 XL-B1010RGBT-HF, U33 XL-B1010RGBT-HF, U34 XL-B1010RGBT-HF, U35 XL-B1010RGBT-HF, U36 XL-B1010RGBT-HF, U37 XL-B1010RGBT-HF, U38 XL-B1010RGBT-HF, U39 XL-B1010RGBT-HF, U4 XL-B1010RGBT-HF, U40 XL-B1010RGBT-HF, U41 XL-B1010RGBT-HF, U42 XL-B1010RGBT-HF, U43 XL-B1010RGBT-HF, U44 XL-B1010RGBT-HF, U45 XL-B1010RGBT-HF, U46 XL-B1010RGBT-HF, U47 XL-B1010RGBT-HF, U48 XL-B1010RGBT-HF, U49 XL-B1010RGBT-HF, U5 XL-B1010RGBT-HF, U50 XL-B1010RGBT-HF, U51 XL-B1010RGBT-HF, U52 XL-B1010RGBT-HF, U53 XL-B1010RGBT-HF, U54 XL-B1010RGBT-HF, U55 XL-B1010RGBT-HF, U56 XL-B1010RGBT-HF, U57 XL-B1010RGBT-HF, U58 XL-B1010RGBT-HF, U59 XL-B1010RGBT-HF, U6 XL-B1010RGBT-HF, U60 XL-B1010RGBT-HF, U61 XL-B1010RGBT-HF, U62 XL-B1010RGBT-HF, U63 XL-B1010RGBT-HF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

Commit message: Matrix design, visual
Parts:
- moved CN3 0.27 mm to (113.6, 60.0)
- moved CN4 0.27 mm to (92.4, 60.0)
- moved U10 0.27 mm to (91.0, 68.0)
- moved U100 0.27 mm to (109.0, 62.0)
- moved U101 0.27 mm to (113.0, 64.0)
- moved U102 0.27 mm to (111.0, 64.0)
- moved U103 0.27 mm to (109.0, 64.0)
- moved U104 0.27 mm to (113.0, 66.0)
- moved U105 0.27 mm to (111.0, 66.0)
- moved U106 0.27 mm to (109.0, 66.0)
- moved U107 0.27 mm to (113.0, 68.0)
- moved U108 0.27 mm to (111.0, 68.0)
- moved U109 0.27 mm to (109.0, 68.0)
- moved U11 0.27 mm to (93.0, 52.0)
- moved U110 0.27 mm to (115.0, 52.0)
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Connections:
- CN3 pad 10: unconnected-(CN3-Pad10) -> GND
- CN3 pad 11: unconnected-(CN3-Pad11) -> GND
- CN3 pad 12: unconnected-(CN3-Pad12) -> GND
- CN3 pad 13: unconnected-(CN3-Pad13) -> GND
- CN3 pad 14: unconnected-(CN3-Pad14) -> GND
- CN3 pad 15: unconnected-(CN3-Pad15) -> GND
- CN3 pad 16: unconnected-(CN3-Pad16) -> GND
- CN3 pad 17: unconnected-(CN3-Pad17) -> GND
- CN3 pad 18: unconnected-(CN3-Pad18) -> GND
- CN3 pad 19: unconnected-(CN3-Pad19) -> GND
- CN3 pad 20: unconnected-(CN3-Pad20) -> GND
- CN3 pad 4: unconnected-(CN3-Pad4) -> GND
- CN3 pad 5: unconnected-(CN3-Pad5) -> GND
- CN3 pad 6: unconnected-(CN3-Pad6) -> GND
- CN3 pad 7: unconnected-(CN3-Pad7) -> GND
- CN3 pad 8: unconnected-(CN3-Pad8) -> GND
- CN3 pad 9: unconnected-(CN3-Pad9) -> GND
- CN4 pad 24: unconnected-(CN4-Pad24) -> GND
- CN4 pad 25: unconnected-(CN4-Pad25) -> GND
- CN4 pad 26: unconnected-(CN4-Pad26) -> GND
- CN4 pad 27: unconnected-(CN4-Pad27) -> GND
- CN4 pad 29: unconnected-(CN4-Pad29) -> GND
- CN4 pad 30: unconnected-(CN4-Pad30) -> GND
- CN4 pad 31: unconnected-(CN4-Pad31) -> GND
- CN4 pad 32: unconnected-(CN4-Pad32) -> GND
- CN4 pad 5: unconnected-(CN4-Pad5) -> GND
- CN4 pad 6: unconnected-(CN4-Pad6) -> GND
- CN4 pad 7: unconnected-(CN4-Pad7) -> GND
Routing:
- net SW1: track 30.6 -> 34.6 mm
- net GND: vias 0 -> 24
- added copper zone on B.Cu, net GND
- added copper zone on F.Cu, net GND
- added copper zone on In1.Cu, net GND
- added copper zone on In2.Cu, net GND
Other:
- board text added: "13x9 RGB LED matrix"
- board text added: "EDrTech"
- board text added: "ILM139CM"
- board text added: "v0.1.0"
