File: pcb_src/ILM139C_driver/ILM139C.kicad_sch (KiCad schematic)
At the start: 170 parts, among them CN3 AXE640124D, CN4 AXE640124D, CN5 AXE540127D, CN6 AXE540127D, U1 IS31FL3741A-QFLS4-TR, U10 XL-B1010RGBT-HF, U100 XL-B1010RGBT-HF, U101 XL-B1010RGBT-HF, U102 XL-B1010RGBT-HF, U103 XL-B1010RGBT-HF, U104 XL-B1010RGBT-HF, U105 XL-B1010RGBT-HF, U106 XL-B1010RGBT-HF, U107 XL-B1010RGBT-HF, U108 XL-B1010RGBT-HF, U109 XL-B1010RGBT-HF, U11 XL-B1010RGBT-HF, U110 XL-B1010RGBT-HF, U111 XL-B1010RGBT-HF, U112 XL-B1010RGBT-HF, U113 XL-B1010RGBT-HF, U114 XL-B1010RGBT-HF, U115 XL-B1010RGBT-HF, U116 XL-B1010RGBT-HF, U117 XL-B1010RGBT-HF, U118 XL-B1010RGBT-HF, U12 XL-B1010RGBT-HF, U13 XL-B1010RGBT-HF, U14 XL-B1010RGBT-HF, U15 XL-B1010RGBT-HF, U16 XL-B1010RGBT-HF, U17 XL-B1010RGBT-HF, U18 XL-B1010RGBT-HF, U19 XL-B1010RGBT-HF, U2 XL-B1010RGBT-HF, U20 XL-B1010RGBT-HF, U21 XL-B1010RGBT-HF, U22 XL-B1010RGBT-HF, U23 XL-B1010RGBT-HF, U24 XL-B1010RGBT-HF, U25 XL-B1010RGBT-HF, U26 XL-B1010RGBT-HF, U27 XL-B1010RGBT-HF, U28 XL-B1010RGBT-HF, U29 XL-B1010RGBT-HF, U3 XL-B1010RGBT-HF, U30 XL-B1010RGBT-HF, U31 XL-B1010RGBT-HF, U32 XL-B1010RGBT-HF, U33 XL-B1010RGBT-HF, U34 XL-B1010RGBT-HF, U35 XL-B1010RGBT-HF, U36 XL-B1010RGBT-HF, U37 XL-B1010RGBT-HF, U38 XL-B1010RGBT-HF, U39 XL-B1010RGBT-HF, U4 XL-B1010RGBT-HF, U40 XL-B1010RGBT-HF, U41 XL-B1010RGBT-HF, U42 XL-B1010RGBT-HF, U43 XL-B1010RGBT-HF, U44 XL-B1010RGBT-HF, U45 XL-B1010RGBT-HF, U46 XL-B1010RGBT-HF, U47 XL-B1010RGBT-HF, U48 XL-B1010RGBT-HF, U49 XL-B1010RGBT-HF, U5 XL-B1010RGBT-HF, U50 XL-B1010RGBT-HF, U51 XL-B1010RGBT-HF, U52 XL-B1010RGBT-HF, U53 XL-B1010RGBT-HF, U54 XL-B1010RGBT-HF, U55 XL-B1010RGBT-HF, U56 XL-B1010RGBT-HF, U57 XL-B1010RGBT-HF, U58 XL-B1010RGBT-HF, U59 XL-B1010RGBT-HF, U6 XL-B1010RGBT-HF, U60 XL-B1010RGBT-HF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

Commit message: Added driver module
Parts:
- removed CN3, CN4: AXE640124D, easyeda2kicad:CONN-SMD_40P-P0.40_OK-14GM040-04, symbol easyeda2kicad:AXE640124D
- removed U10, U100, U101, U102, U103, U104, U105, U106, U107, U108, U109, U11, U110, U111, U112, U113, U114, U115, U116, U117, U118, U12, U13, U14, U15, U16, U17, U18, U19, U2, U20, U21, U22, U23, U24, U25, U26, U27, U28, U29, U3, U30, U31, U32, U33, U34, U35, U36, U37, U38, U39, U4, U40, U41, U42, U43, U44, U45, U46, U47, U48, U49, U5, U50, U51, U52, U53, U54, U55, U56, U57, U58, U59, U6, U60, U61, U62, U63, U64, U65, U66, U67, U68, U69, U7, U70, U71, U72, U73, U74, U75, U76, U77, U78, U79, U8, U80, U81, U82, U83, U84, U85, U86, U87, U88, U89, U9, U90, U91, U92, U93, U94, U95, U96, U97, U98, U99: XL-B1010RGBT-HF, easyeda2kicad:LED-SMD_4P-L1.0-W1.0-TR_1, symbol easyeda2kicad:XL-B1010RGBT-HF
- added CN1, CN2: HC-1.0-2PWT, easyeda2kicad:CONN-SMD_HC-1.0-2PWT, symbol easyeda2kicad:HC-1.0-2PWT
- added R42, R43, R44, R45, R46: 0, Resistor_SMD:R_0603_1608Metric, symbol Device:R
- added TP1, TP2, TP3: TestPoint, TestPoint:TestPoint_Pad_D1.0mm, symbol Connector:TestPoint
- added U2, U3: HC-1.0-4PWT-B-HW, easyeda2kicad:CONN-SMD_4P-P1.00_HCTL_HC-1.0-4PWT, symbol easyeda2kicad:HC-1.0-4PWT-B-HW
Connections:
- net GND: now also CN5.10, CN5.12, CN5.14, CN5.16, CN5.18, CN5.20, CN5.22, CN5.24, CN5.26, CN5.28, CN5.30, CN5.32, CN5.34, CN5.36, CN5.38, CN5.40, CN5.8, CN6.10, CN6.12, CN6.14, CN6.17, CN6.19, CN6.21, CN6.23, CN6.27, CN6.29, CN6.31, CN1.2, CN1.3, CN1.4, CN2.2, CN2.3, CN2.4, R42.2, TP2.1, U2.4, U2.5, U2.6, U3.4, U3.5, U3.6; no longer U1.8 (ADDR)
- net INTB: now also TP3.1
- net SCL: now also R43.2, U2.1, U3.1
- net SDA: now also R44.2, U2.2, U3.2
- net SDB: now also TP1.1
- net VCC: now also CN1.1, CN2.1, R45.2, R46.1
- new net: R42.1, R43.1, R44.1, R45.1, U1.8 (ADDR)
- new net 3V3: R46.2, U2.3, U3.3
Other:
- note added: "3V3 -> VCC JUMPER"
- note added: "INTERRUPT PIN (USE EXTERNAL PULL UP IF IN USE)"
- note added: "POWER CONNECTORS (2.7V-5.5V)"
- note added: "QWIIC CONNECTORS"
- note added: "SHUTDOWN PIN (CONNECT TO GND TO SHUT DOWN)"
- company: (none) -> EDrTech d.o.o.
- title: (none) -> ILM139CD
- moved on the sheet: C1, C2, C3, C4, C5, C6, C7, CN5, CN6, R1, R10, R11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

Commit message: QWIIC things added
Parts:
- added G1: qwiic_Logo, easyeda2kicad:qwiic_3mm, symbol easyeda2kicad:qwiic_Logo
Other:
- note added: "CONNECTORS"
- note removed: "QWIIC CONNECTORS"
Changed lines of the file:
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@@
 		)
 	)
-	(text "QWIIC CONNECTORS"
+	(text "CONNECTORS"
 		(exclude_from_sim no)
-		(at 73.152 150.114 0)
+		(at 80.772 150.114 0)
 		(effects
 			(font
@@
 					(unit 1)
 				)
+			)
+		)
+	)
+	(symbol
+		(lib_id "easyeda2kicad:qwiic_Logo")
+		(at 64.77 149.86 0)
+		(unit 1)
+		(exclude_from_sim no)
+		(in_bom yes)
+		(on_board no)
+		(dnp no)
+		(fields_autoplaced yes)
+		(property "Reference" "G1"
+			(at 64.77 146.05 0)
+			(effects
+				(font
+					(size 1.27 1.27)
+				)
+				(hide yes)
+			)
+		)
+		(property "Value" "qwiic_Logo"
+			(at 64.77 153.67 0)
+			(effects
+				(font
+					(size 1.27 1.27)
+				)
+				(hide yes)
+			)
+		)
+		(property "Footprint" "easyeda2kicad:qwiic_3mm"
+			(at 64.77 156.21 0)
+			(effects
+				(font
+					(size 1.27 1.27)
+				)
+				(hide yes)
+			)
+		)
+		(property "Datasheet" ""
+			(at 64.77 149.86 0)
+			(effects
+				(font
+					(size 1.27 1.27)
+				)
+				(hide yes)
+			)
+		)
+		(property "Description" ""
+			(at 64.77 149.86 0)
+			(effects
+				(font
+					(size 1.27 1.27)
+				)
+				(hide yes)
+			)
+		)
+		(instances
+			(project ""
+				(path "/65360ab6-4927-4267-9a36-4076d5b6b08f"
+					(reference "G1")
+					(unit 1)
+				)

Commit message: Added pinout, fixed qwiic
Connections:
- net 3V3: now also U2.2, U3.2; no longer U2.3, U3.3
- net GND: now also U2.1, U3.1; no longer U2.4, U3.4
- net SCL: now also U2.4, U3.4; no longer U2.1, U3.1
- net SDA: now also U2.3, U3.3; no longer U2.2, U3.2
