File: pcb_src/v1.0.1./ILM139C_driver/ILM139C.kicad_pcb (KiCad board)
At the start: 4 copper layers, 26 x 18 mm, 64 parts, among them CN1 HC-1.0-2PWT, CN2 HC-1.0-2PWT, CN5 AXE540127D, CN6 AXE540127D, U1 IS31FL3741A-QFLS4-TR, U2 HC-1.0-4PWT-B-HW, U3 HC-1.0-4PWT-B-HW

Commit message: Updated to latest version
Parts:
- removed R46: 0, Resistor_SMD:R_0603_1608Metric
- added C10: 22uF, Capacitor_SMD:C_0805_2012Metric, B.Cu at (97.6, 62.0)
- added C11: 22uF, Capacitor_SMD:C_0603_1608Metric, B.Cu at (97.8, 63.9)
- added C8: 22uF, Capacitor_SMD:C_0805_2012Metric, B.Cu at (97.6, 58.0)
- added C9: 22uF, Capacitor_SMD:C_0805_2012Metric, B.Cu at (97.6, 60.0)
- added G***: LOGO, easyeda2kicad:qwiic_3mm, B.Cu at (92.6, 60.9)
- added G***: LOGO, LOGO, B.Cu at (104.1, 71.0)
- added JP1: Jumper_2_Bridged, Jumper:SolderJumper-2_P1.3mm_Bridged2Bar_RoundedPad1.0x1.5mm, B.Cu at (98.3, 67.1)
- added U4: BTC-3215-BN02, easyeda2kicad:SMD-1_L3.0-W2.0-H1.5, B.Cu at (104.7, 59.2)
- added U5: BTC-3215-BN02, easyeda2kicad:SMD-1_L3.0-W2.0-H1.5, B.Cu at (101.8, 63.0)
- added U6: BTC-3215-BN02, easyeda2kicad:SMD-1_L3.0-W2.0-H1.5, B.Cu at (101.3, 59.7)
- added U7: BTC-3215-BN02, easyeda2kicad:SMD-1_L3.0-W2.0-H1.5, B.Cu at (105.2, 62.5)
- moved TP1 4.10 mm to (106.7, 52.9)
- moved TP2 4.10 mm to (104.7, 52.9)
- moved TP3 4.10 mm to (108.7, 52.9)
Routing:
- net SCL: track 39.5 -> 32.7 mm, vias 3 -> 2
- net SDA: track 39.5 -> 33.5 mm, vias 3 -> 2
- net INTB: track 5.72 -> 9.08 mm, vias 2 -> 1
- net VCC: track 46.5 -> 49.7 mm
- net SDB: track 9.42 -> 12.2 mm
- net S39: track 13.9 -> 15.1 mm
- net CS2: track 6.54 -> 7.10 mm
- net CS21: track 7.35 -> 6.93 mm, vias 2 -> 0
- net GND: vias 260 -> 279
Other:
- board text added: "J0"
- board text removed: "EDrTech"
