File: pcb_src/v1.0.1./ILM139C_driver/ILM139C.kicad_sch (KiCad schematic)
At the start: 66 parts, among them CN1 HC-1.0-2PWT, CN2 HC-1.0-2PWT, CN5 AXE540127D, CN6 AXE540127D, U1 IS31FL3741A-QFLS4-TR, U2 HC-1.0-4PWT-B-HW, U3 HC-1.0-4PWT-B-HW

Commit message: Updated to latest version
Parts:
- removed R46: 0, Resistor_SMD:R_0603_1608Metric, symbol Device:R
- added C10: 22uF, Capacitor_SMD:C_0805_2012Metric, symbol Device:C
- added C11: 22uF, Capacitor_SMD:C_0603_1608Metric, symbol Device:C
- added JP1: Jumper_2_Bridged, Jumper:SolderJumper-2_P1.3mm_Bridged2Bar_RoundedPad1.0x1.5mm, symbol Jumper:Jumper_2_Bridged
- added U4, U5, U6, U7: BTC-3215-BN02, easyeda2kicad:SMD-1_L3.0-W2.0-H1.5, symbol easyeda2kicad_n:BTC-3215-BN02
- C8, C9: footprint Capacitor_SMD:C_0603_1608Metric -> Capacitor_SMD:C_0805_2012Metric
Connections:
- net 3V3: now also JP1.1 (A)
- net GND: now also C8.2, C9.2, C10.2, C11.2, U4.1, U5.1, U6.1, U7.1
- net VCC: now also C8.1, C9.1, C10.1, C11.1, JP1.2 (B)
